File: buttons/buttons2.sch (EAGLE design)
At the start: 14 parts, among them U1 TINY2313

Commit message: I think I have a workable Cherry MX design
Parts:
- U$1: value TINY2313 -> TINY2313-*P*
- renumbered U1 to U$1
Changed lines of the file:
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@@
 </classes>
 <parts>
-<part name="U1" library="avr-6" deviceset="TINY2313*" device="-*P*" value="TINY2313"/>
 <part name="SV1" library="con-harting-ml" deviceset="ML26" device="" value="RPi_GPIO"/>
 <part name="JP1" library="SparkFun-Connectors" deviceset="M08" device="1X08" value="LCD_CONN"/>
@@
 <part name="GND5" library="supply1" deviceset="GND" device=""/>
 <part name="GND6" library="supply1" deviceset="GND" device=""/>
+<part name="U$1" library="avr-6" deviceset="TINY2313*" device="-*P*"/>
 </parts>
 <sheets>
@@
 </plain>
 <instances>
-<instance part="U1" gate="G$1" x="111.76" y="86.36"/>
 <instance part="SV1" gate="1" x="35.56" y="78.74"/>
 <instance part="JP1" gate="G$1" x="38.1" y="33.02"/>
@@
 <instance part="GND5" gate="1" x="193.04" y="40.64"/>
 <instance part="GND6" gate="1" x="213.36" y="40.64"/>
+<instance part="U$1" gate="G$1" x="111.76" y="86.36"/>
 </instances>
 <busses>
@@
 <net name="GND" class="0">
 <segment>
-<pinref part="U1" gate="G$1" pin="GND"/>
 <pinref part="C1" gate="G$1" pin="2"/>
+<pinref part="GND7" gate="1" pin="GND"/>
 <wire x1="91.44" y1="58.42" x2="83.82" y2="58.42" width="0.1524" layer="91"/>
-<pinref part="GND7" gate="1" pin="GND"/>
 <wire x1="83.82" y1="58.42" x2="76.2" y2="58.42" width="0.1524" layer="91"/>
 <wire x1="76.2" y1="58.42" x2="76.2" y2="55.88" width="0.1524" layer="91"/>
 <junction x="83.82" y="58.42"/>
+<pinref part="U$1" gate="G$1" pin="GND"/>
+<junction x="91.44" y="58.42"/>
 </segment>
 <segment>
@@
 <net name="N$1" class="0">
 <segment>
-<pinref part="U1" gate="G$1" pin="(OC1B)PB4"/>
 <wire x1="129.54" y1="93.98" x2="170.18" y2="93.98" width="0.1524" layer="91"/>
 <wire x1="170.18" y1="93.98" x2="170.18" y2="81.28" width="0.1524" layer="91"/>
 <pinref part="S6" gate="G$1" pin="PIN-1"/>
+<pinref part="U$1" gate="G$1" pin="(OC1B)PB4"/>
 </segment>
 </net>
 <net name="N$2" class="0">
 <segment>
-<pinref part="U1" gate="G$1" pin="(OC1A)PB3"/>
 <wire x1="129.54" y1="91.44" x2="193.04" y2="91.44" width="0.1524" layer="91"/>
 <pinref part="S5" gate="G$1" pin="PIN-1"/>
 <wire x1="193.04" y1="91.44" x2="193.04" y2="81.28" width="0.1524" layer="91"/>
+<pinref part="U$1" gate="G$1" pin="(OC1A)PB3"/>
 </segment>
 </net>
 <net name="N$3" class="0">
 <segment>
-<pinref part="U1" gate="G$1" pin="(OC0A)PB2"/>
 <wire x1="129.54" y1="88.9" x2="213.36" y2="88.9" width="0.1524" layer="91"/>
 <pinref part="S4" gate="G$1" pin="PIN-1"/>
 <wire x1="213.36" y1="88.9" x2="213.36" y2="81.28" width="0.1524" layer="91"/>
+<pinref part="U$1" gate="G$1" pin="(OC0A)PB2"/>
 </segment>
 </net>
 <net name="N$4" class="0">
 <segment>
-<pinref part="U1" gate="G$1" pin="(AIN1)PB1"/>
 <wire x1="129.54" y1="86.36" x2="162.56" y2="86.36" width="0.1524" layer="91"/>
 <wire x1="162.56" y1="86.36" x2="162.56" y2="63.5" width="0.1524" layer="91"/>
@@
 <pinref part="S3" gate="G$1" pin="PIN-1"/>
 <wire x1="170.18" y1="63.5" x2="170.18" y2="55.88" width="0.1524" layer="91"/>
+<pinref part="U$1" gate="G$1" pin="(AIN1)PB1"/>
 </segment>
 </net>
 <net name="N$5" class="0">
 <segment>
-<pinref part="U1" gate="G$1" pin="(AIN0)PB0"/>
 <wire x1="129.54" y1="83.82" x2="160.02" y2="83.82" width="0.1524" layer="91"/>
 <wire x1="160.02" y1="83.82" x2="160.02" y2="66.04" width="0.1524" layer="91"/>
@@
 <pinref part="S2" gate="G$1" pin="PIN-1"/>
 <wire x1="193.04" y1="66.04" x2="193.04" y2="55.88" width="0.1524" layer="91"/>
+<pinref part="U$1" gate="G$1" pin="(AIN0)PB0"/>
 </segment>
 </net>
 <net name="N$6" class="0">
 <segment>
-<pinref part="U1" gate="G$1" pin="(ICP)PD6"/>
 <wire x1="129.54" y1="73.66" x2="157.48" y2="73.66" width="0.1524" layer="91"/>
 <wire x1="157.48" y1="73.66" x2="157.48" y2="68.58" width="0.1524" layer="91"/>
@@
 <pinref part="S1" gate="G$1" pin="PIN-1"/>
 <wire x1="213.36" y1="68.58" x2="213.36" y2="55.88" width="0.1524" layer="91"/>
+<pinref part="U$1" gate="G$1" pin="(ICP)PD6"/>
 </segment>
 </net>
 <net name="VCC" class="0">
 <segment>
-<pinref part="U1" gate="G$1" pin="VCC"/>
 <pinref part="C1" gate="G$1" pin="1"/>
+<pinref part="P+1" gate="VCC" pin="VCC"/>
 <wire x1="91.44" y1="66.04" x2="83.82" y2="66.04" width="0.1524" layer="91"/>
-<pinref part="P+1" gate="VCC" pin="VCC"/>
 <wire x1="83.82" y1="66.04" x2="76.2" y2="66.04" width="0.1524" layer="91"/>
 <wire x1="76.2" y1="66.04" x2="76.2" y2="68.58" width="0.1524" layer="91"/>
 <junction x="83.82" y="66.04"/>
+<pinref part="U$1" gate="G$1" pin="VCC"/>
+<junction x="91.44" y="66.04"/>
 </segment>
 <segment>
@@
 </segment>
 <segment>
-<pinref part="U1" gate="G$1" pin="(RXD)PD0"/>
 <wire x1="129.54" y1="58.42" x2="139.7" y2="58.42" width="0.1524" layer="91"/>
 <label x="137.16" y="58.42" size="1.778" layer="95"/>
+<pinref part="U$1" gate="G$1" pin="(RXD)PD0"/>
 </segment>
 </net>
 <net name="BUTTON2" class="0">
 <segment>
-<pinref part="U1" gate="G$1" pin="(TXD)PD1"/>
 <wire x1="129.54" y1="60.96" x2="139.7" y2="60.96" width="0.1524" layer="91"/>
 <label x="137.16" y="60.96" size="1.778" layer="95"/>
+<pinref part="U$1" gate="G$1" pin="(TXD)PD1"/>
 </segment>
 <segment>
@@
 <net name="BUTTON3" class="0">
 <segment>
-<pinref part="U1" gate="G$1" pin="PA1(XTAL2)"/>
+<label x="76.2" y="81.28" size="1.778" layer="95"/>
+<pinref part="U$1" gate="G$1" pin="PA1(XTAL2)"/>
 <wire x1="91.44" y1="81.28" x2="83.82" y2="81.28" width="0.1524" layer="91"/>
-<label x="76.2" y="81.28" size="1.778" layer="95"/>
+<junction x="91.44" y="81.28"/>
 </segment>
 <segment>
@@
 <net name="BUTTON4" class="0">
 <segment>
-<pinref part="U1" gate="G$1" pin="PA0(XTAL1)"/>
+<label x="76.2" y="76.2" size="1.778" layer="95"/>
+<pinref part="U$1" gate="G$1" pin="PA0(XTAL1)"/>
 <wire x1="91.44" y1="76.2" x2="83.82" y2="76.2" width="0.1524" layer="91"/>
-<label x="76.2" y="76.2" size="1.778" layer="95"/>
+<junction x="91.44" y="76.2"/>
 </segment>
 <segment>
@@
 <net name="BUTTON5" class="0">
 <segment>
-<pinref part="U1" gate="G$1" pin="(INT0)PD2"/>
 <wire x1="129.54" y1="63.5" x2="139.7" y2="63.5" width="0.1524" layer="91"/>
 <label x="137.16" y="63.5" size="1.778" layer="95"/>
+<pinref part="U$1" gate="G$1" pin="(INT0)PD2"/>
 </segment>
 <segment>
@@
 <net name="BUTTON6" class="0">
 <segment>
-<pinref part="U1" gate="G$1" pin="(INT1)PD3"/>
 <wire x1="129.54" y1="66.04" x2="139.7" y2="66.04" width="0.1524" layer="91"/>
 <label x="137.16" y="66.04" size="1.778" layer="95"/>
-</segment>
-<segment>
+<pinref part="U$1" gate="G$1" pin="(INT1)PD3"/>
+</segment>
+<segment>

Commit message: more work on button PCB, but not done
Problem is that the buttons need to be rotated
180 degrees!  Because the board will be flipped,
the top of the PCB will be towards the bottom
of the top plate of the enclosure.  Duh.
Parts:
- U1: value TINY2313-*P* -> attiny2313
- renumbered U$1 to U1
Changed lines of the file:
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@@
 <part name="GND5" library="supply1" deviceset="GND" device=""/>
 <part name="GND6" library="supply1" deviceset="GND" device=""/>
-<part name="U$1" library="avr-6" deviceset="TINY2313*" device="-*P*"/>
+<part name="U1" library="avr-6" deviceset="TINY2313*" device="-*P*" value="attiny2313"/>
 </parts>
 <sheets>
@@
 <instance part="GND5" gate="1" x="193.04" y="40.64"/>
 <instance part="GND6" gate="1" x="213.36" y="40.64"/>
-<instance part="U$1" gate="G$1" x="111.76" y="86.36"/>
+<instance part="U1" gate="G$1" x="111.76" y="86.36"/>
 </instances>
 <busses>
@@
 <wire x1="76.2" y1="58.42" x2="76.2" y2="55.88" width="0.1524" layer="91"/>
 <junction x="83.82" y="58.42"/>
-<pinref part="U$1" gate="G$1" pin="GND"/>
+<pinref part="U1" gate="G$1" pin="GND"/>
 <junction x="91.44" y="58.42"/>
 </segment>
@@
 <wire x1="170.18" y1="93.98" x2="170.18" y2="81.28" width="0.1524" layer="91"/>
 <pinref part="S6" gate="G$1" pin="PIN-1"/>
-<pinref part="U$1" gate="G$1" pin="(OC1B)PB4"/>
+<pinref part="U1" gate="G$1" pin="(OC1B)PB4"/>
 </segment>
 </net>
@@
 <pinref part="S5" gate="G$1" pin="PIN-1"/>
 <wire x1="193.04" y1="91.44" x2="193.04" y2="81.28" width="0.1524" layer="91"/>
-<pinref part="U$1" gate="G$1" pin="(OC1A)PB3"/>
+<pinref part="U1" gate="G$1" pin="(OC1A)PB3"/>
 </segment>
 </net>
@@
 <pinref part="S4" gate="G$1" pin="PIN-1"/>
 <wire x1="213.36" y1="88.9" x2="213.36" y2="81.28" width="0.1524" layer="91"/>
-<pinref part="U$1" gate="G$1" pin="(OC0A)PB2"/>
+<pinref part="U1" gate="G$1" pin="(OC0A)PB2"/>
 </segment>
 </net>
@@
 <pinref part="S3" gate="G$1" pin="PIN-1"/>
 <wire x1="170.18" y1="63.5" x2="170.18" y2="55.88" width="0.1524" layer="91"/>
-<pinref part="U$1" gate="G$1" pin="(AIN1)PB1"/>
+<pinref part="U1" gate="G$1" pin="(AIN1)PB1"/>
 </segment>
 </net>
@@
 <pinref part="S2" gate="G$1" pin="PIN-1"/>
 <wire x1="193.04" y1="66.04" x2="193.04" y2="55.88" width="0.1524" layer="91"/>
-<pinref part="U$1" gate="G$1" pin="(AIN0)PB0"/>
+<pinref part="U1" gate="G$1" pin="(AIN0)PB0"/>
 </segment>
 </net>
@@
 <pinref part="S1" gate="G$1" pin="PIN-1"/>
 <wire x1="213.36" y1="68.58" x2="213.36" y2="55.88" width="0.1524" layer="91"/>
-<pinref part="U$1" gate="G$1" pin="(ICP)PD6"/>
+<pinref part="U1" gate="G$1" pin="(ICP)PD6"/>
 </segment>
 </net>
@@
 <wire x1="76.2" y1="66.04" x2="76.2" y2="68.58" width="0.1524" layer="91"/>
 <junction x="83.82" y="66.04"/>
-<pinref part="U$1" gate="G$1" pin="VCC"/>
+<pinref part="U1" gate="G$1" pin="VCC"/>
 <junction x="91.44" y="66.04"/>
 </segment>
@@
 <wire x1="129.54" y1="58.42" x2="139.7" y2="58.42" width="0.1524" layer="91"/>
 <label x="137.16" y="58.42" size="1.778" layer="95"/>
-<pinref part="U$1" gate="G$1" pin="(RXD)PD0"/>
+<pinref part="U1" gate="G$1" pin="(RXD)PD0"/>
 </segment>
 </net>
@@
 <wire x1="129.54" y1="60.96" x2="139.7" y2="60.96" width="0.1524" layer="91"/>
 <label x="137.16" y="60.96" size="1.778" layer="95"/>
-<pinref part="U$1" gate="G$1" pin="(TXD)PD1"/>
+<pinref part="U1" gate="G$1" pin="(TXD)PD1"/>
 </segment>
 <segment>
@@
 <segment>
 <label x="76.2" y="81.28" size="1.778" layer="95"/>
-<pinref part="U$1" gate="G$1" pin="PA1(XTAL2)"/>
+<pinref part="U1" gate="G$1" pin="PA1(XTAL2)"/>
 <wire x1="91.44" y1="81.28" x2="83.82" y2="81.28" width="0.1524" layer="91"/>
 <junction x="91.44" y="81.28"/>
@@
 <segment>
 <label x="76.2" y="76.2" size="1.778" layer="95"/>
-<pinref part="U$1" gate="G$1" pin="PA0(XTAL1)"/>
+<pinref part="U1" gate="G$1" pin="PA0(XTAL1)"/>
 <wire x1="91.44" y1="76.2" x2="83.82" y2="76.2" width="0.1524" layer="91"/>
 <junction x="91.44" y="76.2"/>
@@
 <wire x1="129.54" y1="63.5" x2="139.7" y2="63.5" width="0.1524" layer="91"/>
 <label x="137.16" y="63.5" size="1.778" layer="95"/>
-<pinref part="U$1" gate="G$1" pin="(INT0)PD2"/>
+<pinref part="U1" gate="G$1" pin="(INT0)PD2"/>
 </segment>
 <segment>
@@
 <wire x1="129.54" y1="66.04" x2="139.7" y2="66.04" width="0.1524" layer="91"/>
 <label x="137.16" y="66.04" size="1.778" layer="95"/>
-<pinref part="U$1" gate="G$1" pin="(INT1)PD3"/>
-</segment>
-<segment>
+<pinref part="U1" gate="G$1" pin="(INT1)PD3"/>
+</segment>
+<segment>

Commit message: finished routing updated buttons2 PCB
This has (I think) adequate clearance for an 18mm x 18mm
keycap: the centers of the switches are 18.5mm apart, hopefully
this is enough room.
Parts:
- removed SV1: RPi_GPIO, con-harting-ml:ML26
- added JP2: LCD_CONN, SparkFun-Connectors:M081X08
- JP1: value LCD_CONN -> RPi_GPIO; device SparkFun-Connectors:M081X08 -> con-harting-ml:ML26
Connections:
- net BUTTON1: now also JP1.3; no longer SV1.3
- net BUTTON2: now also JP1.5; no longer SV1.5
- net BUTTON3: now also JP1.7; no longer SV1.7
- net BUTTON4: now also JP1.11; no longer SV1.11
- net BUTTON5: now also JP1.13; no longer SV1.13
- net BUTTON6: now also JP1.15; no longer SV1.15
- net CS: now also JP1.24, JP2.3; no longer JP1.3, SV1.24
- net DC: now also JP1.18, JP2.5; no longer JP1.5, SV1.18
- net GND: now also JP1.25, JP2.2; no longer JP1.2, SV1.25
- net LED: now also JP1.12, JP2.8; no longer JP1.8, SV1.12
- net MOSI: now also JP1.19, JP2.6; no longer JP1.6, SV1.19
- net RESET: now also JP1.22, JP2.4; no longer JP1.4, SV1.22
- net SCK: now also JP1.23, JP2.7; no longer JP1.7, SV1.23
- net VCC: now also JP2.1; no longer SV1.1
Changed lines of the file:
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@@
 </classes>
 <parts>
-<part name="SV1" library="con-harting-ml" deviceset="ML26" device="" value="RPi_GPIO"/>
-<part name="JP1" library="SparkFun-Connectors" deviceset="M08" device="1X08" value="LCD_CONN"/>
+<part name="JP1" library="con-harting-ml" deviceset="ML26" device="" value="RPi_GPIO"/>
+<part name="JP2" library="SparkFun-Connectors" deviceset="M08" device="1X08" value="LCD_CONN"/>
 <part name="C1" library="capacitor-wima" deviceset="C" device="2.5/2" value="0.1uF"/>
 <part name="P+1" library="supply1" deviceset="VCC" device=""/>
@@
 </plain>
 <instances>
-<instance part="SV1" gate="1" x="35.56" y="78.74"/>
-<instance part="JP1" gate="G$1" x="38.1" y="33.02"/>
+<instance part="JP1" gate="1" x="35.56" y="78.74"/>
+<instance part="JP2" gate="G$1" x="38.1" y="33.02"/>
 <instance part="C1" gate="G$1" x="83.82" y="63.5"/>
 <instance part="P+1" gate="VCC" x="76.2" y="71.12"/>
@@
 </segment>
 <segment>
-<pinref part="JP1" gate="G$1" pin="2"/>
+<pinref part="JP2" gate="G$1" pin="2"/>
 <pinref part="GND8" gate="1" pin="GND"/>
 <wire x1="43.18" y1="27.94" x2="58.42" y2="27.94" width="0.1524" layer="91"/>
@@
 </segment>
 <segment>
-<pinref part="SV1" gate="1" pin="25"/>
+<pinref part="JP1" gate="1" pin="25"/>
 <wire x1="43.18" y1="93.98" x2="66.04" y2="93.98" width="0.1524" layer="91"/>
 <wire x1="66.04" y1="93.98" x2="66.04" y2="88.9" width="0.1524" layer="91"/>
@@
 </segment>
 <segment>
-<pinref part="JP1" gate="G$1" pin="1"/>
+<pinref part="JP2" gate="G$1" pin="1"/>
 <pinref part="P+2" gate="VCC" pin="VCC"/>
 <wire x1="43.18" y1="25.4" x2="78.74" y2="25.4" width="0.1524" layer="91"/>
@@
 </segment>
 <segment>
-<pinref part="SV1" gate="1" pin="1"/>
+<pinref part="JP1" gate="1" pin="1"/>
 <wire x1="43.18" y1="63.5" x2="66.04" y2="63.5" width="0.1524" layer="91"/>
 <wire x1="66.04" y1="63.5" x2="66.04" y2="68.58" width="0.1524" layer="91"/>
@@
 <net name="CS" class="0">
 <segment>
-<pinref part="JP1" gate="G$1" pin="3"/>
+<pinref part="JP2" gate="G$1" pin="3"/>
 <wire x1="43.18" y1="30.48" x2="50.8" y2="30.48" width="0.1524" layer="91"/>
 <label x="50.8" y="30.48" size="1.778" layer="95"/>
 </segment>
 <segment>
-<pinref part="SV1" gate="1" pin="24"/>
+<pinref part="JP1" gate="1" pin="24"/>
 <wire x1="27.94" y1="91.44" x2="20.32" y2="91.44" width="0.1524" layer="91"/>
 <label x="17.78" y="91.44" size="1.778" layer="95"/>
@@
 <net name="RESET" class="0">
 <segment>
-<pinref part="JP1" gate="G$1" pin="4"/>
+<pinref part="JP2" gate="G$1" pin="4"/>
 <wire x1="43.18" y1="33.02" x2="50.8" y2="33.02" width="0.1524" layer="91"/>
 <label x="50.8" y="33.02" size="1.778" layer="95"/>
 </segment>
 <segment>
-<pinref part="SV1" gate="1" pin="22"/>
+<pinref part="JP1" gate="1" pin="22"/>
 <wire x1="27.94" y1="88.9" x2="20.32" y2="88.9" width="0.1524" layer="91"/>
 <label x="15.24" y="88.9" size="1.778" layer="95"/>
@@
 <net name="DC" class="0">
 <segment>
-<pinref part="JP1" gate="G$1" pin="5"/>
+<pinref part="JP2" gate="G$1" pin="5"/>
 <wire x1="43.18" y1="35.56" x2="50.8" y2="35.56" width="0.1524" layer="91"/>
 <label x="50.8" y="35.56" size="1.778" layer="95"/>
 </segment>
 <segment>
-<pinref part="SV1" gate="1" pin="18"/>
+<pinref part="JP1" gate="1" pin="18"/>
 <wire x1="27.94" y1="83.82" x2="20.32" y2="83.82" width="0.1524" layer="91"/>
 <label x="17.78" y="83.82" size="1.778" layer="95"/>
@@
 <net name="MOSI" class="0">
 <segment>
-<pinref part="JP1" gate="G$1" pin="6"/>
+<pinref part="JP2" gate="G$1" pin="6"/>
 <wire x1="43.18" y1="38.1" x2="50.8" y2="38.1" width="0.1524" layer="91"/>
 <label x="50.8" y="38.1" size="1.778" layer="95"/>
 </segment>
 <segment>
-<pinref part="SV1" gate="1" pin="19"/>
+<pinref part="JP1" gate="1" pin="19"/>
 <wire x1="43.18" y1="86.36" x2="50.8" y2="86.36" width="0.1524" layer="91"/>
 <label x="48.26" y="86.36" size="1.778" layer="95"/>
@@
 <net name="SCK" class="0">
 <segment>
-<pinref part="JP1" gate="G$1" pin="7"/>
+<pinref part="JP2" gate="G$1" pin="7"/>
 <wire x1="43.18" y1="40.64" x2="50.8" y2="40.64" width="0.1524" layer="91"/>
 <label x="50.8" y="40.64" size="1.778" layer="95"/>
 </segment>
 <segment>
-<pinref part="SV1" gate="1" pin="23"/>
+<pinref part="JP1" gate="1" pin="23"/>
 <wire x1="43.18" y1="91.44" x2="50.8" y2="91.44" width="0.1524" layer="91"/>
 <label x="48.26" y="91.44" size="1.778" layer="95"/>
@@
 <net name="BUTTON1" class="0">
 <segment>
-<pinref part="SV1" gate="1" pin="3"/>
+<pinref part="JP1" gate="1" pin="3"/>
 <wire x1="43.18" y1="66.04" x2="50.8" y2="66.04" width="0.1524" layer="91"/>
 <label x="48.26" y="66.04" size="1.778" layer="95"/>
@@
 </segment>
 <segment>
-<pinref part="SV1" gate="1" pin="5"/>
+<pinref part="JP1" gate="1" pin="5"/>
 <wire x1="43.18" y1="68.58" x2="50.8" y2="68.58" width="0.1524" layer="91"/>
 <label x="48.26" y="68.58" size="1.778" layer="95"/>
@@
 </segment>
 <segment>
-<pinref part="SV1" gate="1" pin="7"/>
+<pinref part="JP1" gate="1" pin="7"/>
 <wire x1="43.18" y1="71.12" x2="50.8" y2="71.12" width="0.1524" layer="91"/>
 <label x="48.26" y="71.12" size="1.778" layer="95"/>
@@
 </segment>
 <segment>
-<pinref part="SV1" gate="1" pin="11"/>
+<pinref part="JP1" gate="1" pin="11"/>
 <wire x1="43.18" y1="76.2" x2="50.8" y2="76.2" width="0.1524" layer="91"/>
 <label x="48.26" y="76.2" size="1.778" layer="95"/>
@@
 </segment>
 <segment>
-<pinref part="SV1" gate="1" pin="13"/>
+<pinref part="JP1" gate="1" pin="13"/>
 <wire x1="43.18" y1="78.74" x2="50.8" y2="78.74" width="0.1524" layer="91"/>
 <label x="48.26" y="78.74" size="1.778" layer="95"/>
@@
 </segment>
 <segment>
-<pinref part="SV1" gate="1" pin="15"/>
+<pinref part="JP1" gate="1" pin="15"/>
 <wire x1="43.18" y1="81.28" x2="50.8" y2="81.28" width="0.1524" layer="91"/>
 <label x="48.26" y="81.28" size="1.778" layer="95"/>
@@
 <net name="LED" class="0">
 <segment>
-<pinref part="JP1" gate="G$1" pin="8"/>
+<pinref part="JP2" gate="G$1" pin="8"/>
 <wire x1="43.18" y1="43.18" x2="50.8" y2="43.18" width="0.1524" layer="91"/>
 <label x="50.8" y="43.18" size="1.778" layer="95"/>
 </segment>
 <segment>
-<pinref part="SV1" gate="1" pin="12"/>
+<pinref part="JP1" gate="1" pin="12"/>
 <wire x1="27.94" y1="76.2" x2="20.32" y2="76.2" width="0.1524" layer="91"/>
 <label x="17.78" y="76.2" size="1.778" layer="95"/>
